File: Electrical/Board_003/mbus_master.sch (KiCad schematic (older format))
At the start: 14 parts, among them J1 Conn_01x02, J2 Conn_01x02, J3 Conn_01x02, Q1 BC337, Q2 BC337, Q3 BC337, Q4 BD136

Commit message: Board_003: Finished Rev A
Parts:
- D1: renamed from 12V1; footprint Diodes_THT:D_A-405_P12.70mm_Horizontal -> Diodes_THT:D_A-405_P7.62mm_Horizontal
- R1, R2, R3, R4, R5, R6: footprint Resistors_THT:R_Axial_DIN0309_L9.0mm_D3.2mm_P12.70mm_Horizontal -> Resistors_THT:R_Axial_DIN0207_L6.3mm_D2.5mm_P10.16mm_Horizontal
Changed lines of the file:
@@
 F 0 "R1" V 3280 6700 50  0000 C CNN
 F 1 "1k" V 3200 6700 50  0000 C CNN
-F 2 "Resistors_THT:R_Axial_DIN0309_L9.0mm_D3.2mm_P12.70mm_Horizontal" V 3130 6700 50  0001 C CNN
+F 2 "Resistors_THT:R_Axial_DIN0207_L6.3mm_D2.5mm_P10.16mm_Horizontal" V 3130 6700 50  0001 C CNN
 F 3 "" H 3200 6700 50  0001 C CNN
 	1    3200 6700
@@
 	3850 6900 3850 7100
 $Comp
-L D_Zener_Small_ALT 12V1
+L D_Zener_Small_ALT D1
 U 1 1 5A6C5A7F
 P 5750 3500
-F 0 "12V1" H 5750 3590 50  0000 C CNN
+F 0 "D1" H 5750 3590 50  0000 C CNN
 F 1 "D_Zener_Small_ALT" H 5750 3410 50  0001 C CNN
-F 2 "Diodes_THT:D_A-405_P12.70mm_Horizontal" V 5750 3500 50  0001 C CNN
+F 2 "Diodes_THT:D_A-405_P7.62mm_Horizontal" V 5750 3500 50  0001 C CNN
 F 3 "" V 5750 3500 50  0001 C CNN
 	1    5750 3500
@@
 F 0 "R6" V 7630 3500 50  0000 C CNN
 F 1 "220k" V 7550 3500 50  0000 C CNN
-F 2 "Resistors_THT:R_Axial_DIN0309_L9.0mm_D3.2mm_P12.70mm_Horizontal" V 7480 3500 50  0001 C CNN
+F 2 "Resistors_THT:R_Axial_DIN0207_L6.3mm_D2.5mm_P10.16mm_Horizontal" V 7480 3500 50  0001 C CNN
 F 3 "" H 7550 3500 50  0001 C CNN
 	1    7550 3500
@@
 F 0 "R5" V 5830 4450 50  0000 C CNN
 F 1 "22k" V 5750 4450 50  0000 C CNN
-F 2 "Resistors_THT:R_Axial_DIN0309_L9.0mm_D3.2mm_P12.70mm_Horizontal" V 5680 4450 50  0001 C CNN
+F 2 "Resistors_THT:R_Axial_DIN0207_L6.3mm_D2.5mm_P10.16mm_Horizontal" V 5680 4450 50  0001 C CNN
 F 3 "" H 5750 4450 50  0001 C CNN
 	1    5750 4450
@@
 F 0 "R4" V 5080 5400 50  0000 C CNN
 F 1 "150" V 5000 5400 50  0000 C CNN
-F 2 "Resistors_THT:R_Axial_DIN0309_L9.0mm_D3.2mm_P12.70mm_Horizontal" V 4930 5400 50  0001 C CNN
+F 2 "Resistors_THT:R_Axial_DIN0207_L6.3mm_D2.5mm_P10.16mm_Horizontal" V 4930 5400 50  0001 C CNN
 F 3 "" H 5000 5400 50  0001 C CNN
 	1    5000 5400
@@
 F 0 "R2" V 4180 4500 50  0000 C CNN
 F 1 "6k8" V 4100 4500 50  0000 C CNN
-F 2 "Resistors_THT:R_Axial_DIN0309_L9.0mm_D3.2mm_P12.70mm_Horizontal" V 4030 4500 50  0001 C CNN
+F 2 "Resistors_THT:R_Axial_DIN0207_L6.3mm_D2.5mm_P10.16mm_Horizontal" V 4030 4500 50  0001 C CNN
 F 3 "" H 4100 4500 50  0001 C CNN
 	1    4100 4500
@@
 F 0 "R3" V 4730 5100 50  0000 C CNN
 F 1 "1" V 4650 5100 50  0000 C CNN
-F 2 "Resistors_THT:R_Axial_DIN0309_L9.0mm_D3.2mm_P12.70mm_Horizontal" V 4580 5100 50  0001 C CNN
+F 2 "Resistors_THT:R_Axial_DIN0207_L6.3mm_D2.5mm_P10.16mm_Horizontal" V 4580 5100 50  0001 C CNN
 F 3 "" H 4650 5100 50  0001 C CNN
 	1    4650 5100
